File: Arm_stepper.kicad_pcb (KiCad board)
At the start: 2 copper layers, 154.5 x 60 mm, 133 parts, among them IC1 L6208D, J1 12V_CONN, J10 ENCODER1, J11 ENCODER2, J3 M1_CONN, J4 Conn_01x06_Male, J5 I2C_CONN, J8 Conn_01x04_Female, J9 USB_B_Mini, M3 MountingHole_3mm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

Commit message: fix
Routing:
- net GNDPWR: track 148.4 -> 283.0 mm
- net GNDD: track 451.9 -> 478.7 mm
Changed lines of the file:
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@@
     (thickness 1.6)
     (drawings 67)
-    (tracks 2012)
+    (tracks 2021)
     (zones 0)
     (modules 133)
@@
   (layers
     (0 F.Cu signal)
-    (31 B.Cu signal hide)
+    (31 B.Cu signal)
     (32 B.Adhes user hide)
     (33 F.Adhes user hide)
@@
   )
   (setup
-    (last_trace_width 0.25)
+    (last_trace_width 3)
     (user_trace_width 0.2)
     (user_trace_width 0.4)
@@
   (via (at 122.1852 116.6584) (size 0.8) (drill 0.4) (layers F.Cu B.Cu) (net 38))
   (segment (start 120.1852 111.95001) (end 110.1852 111.95001) (width 2.5) (layer F.Cu) (net 38))
-  (segment (start 110.1852 113.6584) (end 119.1852 113.6584) (width 2.5) (layer F.Cu) (net 38))
   (segment (start 110.1852 115.6584) (end 119.1852 115.6584) (width 2.5) (layer F.Cu) (net 38))
   (segment (start 120.89359 111.95001) (end 121.1852 111.95001) (width 2.5) (layer F.Cu) (net 38))
@@
   (segment (start 122.1852 116.6584) (end 122.1852 111.95001) (width 2.5) (layer F.Cu) (net 38))
   (segment (start 110.1852 116.6584) (end 122.1852 116.6584) (width 3) (layer F.Cu) (net 38))
+  (segment (start 116 127) (end 116 113.6584) (width 3) (layer F.Cu) (net 38))
+  (segment (start 116 113.6584) (end 119.1852 113.6584) (width 2.5) (layer F.Cu) (net 38))
+  (segment (start 110.1852 113.6584) (end 116 113.6584) (width 2.5) (layer F.Cu) (net 38))
+  (segment (start 164.81 113.8036) (end 164.9952 113.6184) (width 3) (layer F.Cu) (net 38))
+  (segment (start 164.81 126.96) (end 164.81 113.8036) (width 3) (layer F.Cu) (net 38))
   (via (at 89.3064 105.156) (size 0.8) (drill 0.4) (layers F.Cu B.Cu) (net 39))
   (segment (start 89.3304 105.18) (end 89.3064 105.156) (width 0.4) (layer F.Cu) (net 39))
@@
   (via (at 89.2556 98) (size 0.8) (drill 0.4) (layers F.Cu B.Cu) (net 39))
   (segment (start 89.3064 105.156) (end 89.3064 98.0508) (width 0.4) (layer B.Cu) (net 39))
-  (segment (start 138.0656 97.96) (end 171.492 97.96) (width 3) (layer F.Cu) (net 39))
-  (segment (start 124.04 97.96) (end 138.0656 97.96) (width 3) (layer F.Cu) (net 39))
-  (segment (start 124 98) (end 124.04 97.96) (width 3) (layer F.Cu) (net 39))
-  (segment (start 122.682 98) (end 124 98) (width 3) (layer F.Cu) (net 39))
   (segment (start 43.28 98) (end 91.5 98) (width 3.5) (layer F.Cu) (net 39))
   (segment (start 41.91 99.37) (end 43.28 98) (width 3) (layer F.Cu) (net 39))
@@
   (segment (start 46.7 99.37) (end 45.25 99.37) (width 0.25) (layer F.Cu) (net 39))
   (segment (start 46.7 99.37) (end 41.91 99.37) (width 2) (layer F.Cu) (net 39))
+  (segment (start 48.07 98) (end 46.7 99.37) (width 3) (layer B.Cu) (net 39))
+  (segment (start 122.682 98) (end 48.07 98) (width 3) (layer B.Cu) (net 39))
+  (segment (start 45.5 98) (end 45.25 97.75) (width 3) (layer B.Cu) (net 39))
+  (segment (start 48.07 98) (end 45.5 98) (width 3) (layer B.Cu) (net 39))
+  (segment (start 43.53 97.75) (end 41.91 99.37) (width 3) (layer B.Cu) (net 39))
+  (segment (start 45.25 97.75) (end 43.53 97.75) (width 3) (layer B.Cu) (net 39))
+  (segment (start 171.452 98) (end 171.492 97.96) (width 3) (layer B.Cu) (net 39))
+  (segment (start 122.682 98) (end 171.452 98) (width 3) (layer B.Cu) (net 39))
+  (segment (start 122.682 98) (end 173.75 98) (width 3) (layer F.Cu) (net 39))
   (segment (start 77.629001 110.586399) (end 77.629001 111.524403) (width 0.25) (layer F.Cu) (net 40))
   (segment (start 77.629001 111.524403) (end 80.760198 114.6556) (width 0.25) (layer F.Cu) (net 40))
@@
     (connect_pads yes (clearance 0.3))
     (min_thickness 0.254)
-    (fill yes (arc_segments 16) (thermal_gap 0.508) (thermal_bridge_width 0.508) (smoothing fillet) (radius 0.1))
+    (fill yes (arc_segments 16) (thermal_gap 0.508) (thermal_bridge_width 0.508) (smoothing fillet) (radius 1))
     (polygon
       (pts
@@
     (connect_pads yes (clearance 0.3))
     (min_thickness 0.254)
-    (fill yes (arc_segments 16) (thermal_gap 0.508) (thermal_bridge_width 0.508) (smoothing fillet) (radius 0.1))
+    (fill yes (arc_segments 16) (thermal_gap 0.508) (thermal_bridge_width 0.508) (smoothing fillet) (radius 1))
     (polygon
       (pts

Commit message: fixx
Parts:
- moved J1 0.41 mm to (47.1, 99.4)
Changed lines of the file:
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@@
   )
   (setup
-    (last_trace_width 3)
+    (last_trace_width 0.25)
     (user_trace_width 0.2)
     (user_trace_width 0.4)
@@
   )
   (module TerminalBlock_Phoenix:TerminalBlock_Phoenix_PT-1,5-2-3.5-H_1x02_P3.50mm_Horizontal (layer F.Cu)
-    (at 46.7 99.37 270)
+    (at 47.11 99.37 270)
     (descr "Terminal Block Phoenix PT-1,5-2-3.5-H, 2 pins, pitch 3.5mm, size 7x7.6mm^2, drill diamater 1.2mm, pad diameter 2.4mm, see , script-generated using https://github.com/pointhi/kicad-footprint-generator/scripts/TerminalBlock_Phoenix")
     (tags "THT Terminal Block Phoenix PT-1,5-2-3.5-H pitch 3.5mm size 7x7.6mm^2 drill 1.2mm pad 2.4mm")

Commit message: gerber
Parts:
- removed R47: 220, Resistor_SMD:R_0805_2012Metric
Connections:
- C8 pad 2: Net-(C8-Pad2) -> /NRST
- SW1 pad 1: Net-(C8-Pad2) -> /NRST
Routing:
- net Net-(C8-Pad2): track 16.0 -> 0.00 mm
- net /NRST: track 76.0 -> 70.4 mm
