File: Arm_stepper.sch (KiCad schematic (older format))
At the start: 127 parts, among them IC1 L6208D, IC2 L6208D, J1 12V_CONN, J10 ENCODER1, J11 ENCODER2, J2 M1_CONN, J3 M1_CONN, J4 Conn_01x06_Male, J5 I2C_CONN, J6 SWDCONNUSART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

Commit message: gerber
Parts:
- removed R47: 220, Resistor_SMD:R_0805_2012Metric, symbol Device:R
- C12: value 2.2uF -> 4,7uF
Connections:
- net NRST: now also C8.2, SW1.1, SW1.3
Changed lines of the file:
@@
 P 3850 3100
 F 0 "C12" V 3598 3100 50  0000 C CNN
-F 1 "2.2uF" V 3689 3100 50  0000 C CNN
+F 1 "4,7uF" V 3689 3100 50  0000 C CNN
 F 2 "Capacitor_SMD:C_0805_2012Metric" H 3888 2950 50  0001 C CNN
 F 3 "~" H 3850 3100 50  0001 C CNN
@@
 Wire Wire Line
 	4000 2500 4000 2700
-$Comp
-L Device:R R47
-U 1 1 5C476BB5
-P 3300 2500
-F 0 "R47" V 3093 2500 50  0000 C CNN
-F 1 "220" V 3184 2500 50  0000 C CNN
-F 2 "Resistor_SMD:R_0805_2012Metric" V 3230 2500 50  0001 C CNN
-F 3 "~" H 3300 2500 50  0001 C CNN
-	1    3300 2500
-	0    1    1    0
-$EndComp
-Wire Wire Line
-	2600 2500 3150 2500
-Wire Wire Line
-	3450 2500 4000 2500
 Wire Wire Line
 	10700 9200 10850 9200
@@
 Wire Wire Line
 	14850 8050 14850 8350
+Wire Wire Line
+	2600 2500 4000 2500
 $EndSCHEMATC
